File: RRC2021_PCBs/AvionicsBay2_PCB1/RRC2021_PCB1.kicad_pcb (KiCad board)
At the start: 2 copper layers, 114.3 x 73.7 mm, 9 parts, among them U1 ADXL357z, U2 MS5611

Commit message: update
Parts:
- removed GPS1: AULT_GPS, Mounting Holes:1x09
- added C3: 0.1uF, Capacitor_SMD:CP_Elec_3x5.3, F.Cu at (205.7, 74.9)
- added R1: 4.7KOHM-0603-1_10W-1%, Resistors:0603, F.Cu at (204.5, 96.5)
- added R2: 4.7KOHM-0603-1_10W-1%, Resistors:0603, F.Cu at (207.0, 97.8)
- added U3: BN220-GPS, Connector_PinSocket_2.54mm:PinSocket_1x04_P2.54mm_Vertical, F.Cu at (228.6, 102.9)
- added linear_volt_reg2: LM7805_TO220, Package_TO_SOT_THT:TO-220-3_Vertical, F.Cu at (193.0, 80.0)
- moved RF1 32.7 mm to (152.4, 94.0)
Connections:
- RF1 pad 1: Net-(RF1-Pad1) -> (no net)
- RF1 pad 10: Net-(RF1-Pad10) -> (no net)
- RF1 pad 11: Net-(RF1-Pad11) -> (no net)
- RF1 pad 12: Net-(RF1-Pad12) -> (no net)
- RF1 pad 13: Net-(RF1-Pad13) -> (no net)
- RF1 pad 14: Net-(RF1-Pad14) -> (no net)
- RF1 pad 15: Net-(RF1-Pad15) -> (no net)
- RF1 pad 16: Net-(RF1-Pad16) -> (no net)
- RF1 pad 2: Net-(Battery1-Pad2) -> Net-(Battery2-Pad2)
- RF1 pad 3: Net-(RF1-Pad3) -> (no net)
- RF1 pad 4: Net-(C2-Pad1) -> Net-(RF1-Pad4)
- RF1 pad 6: Net-(RF1-Pad6) -> Net-(RF1-Pad4)
- RF1 pad 8: Net-(RF1-Pad8) -> (no net)
- U1 pad 1: Net-(U1-Pad1) -> Net-(R1-Pad2)
- U1 pad 10: Net-(U1-Pad10) -> (no net)
- U1 pad 11: Net-(U1-Pad11) -> (no net)
- U1 pad 12: Net-(U1-Pad12) -> (no net)
- U1 pad 13: Net-(U1-Pad13) -> (no net)
- U1 pad 14: Net-(U1-Pad14) -> (no net)
- U1 pad 3: Net-(U1-Pad3) -> Net-(R2-Pad1)
- U1 pad 4: Net-(U1-Pad4) -> (no net)
- U1 pad 5: Net-(C2-Pad1) -> Net-(R1-Pad1)
- U1 pad 6: Net-(Battery1-Pad2) -> Net-(R1-Pad1)
- U1 pad 8: Net-(U1-Pad8) -> (no net)
- U2 pad 1: Net-(C2-Pad1) -> (no net)
- U2 pad 2: Net-(U1-Pad4) -> (no net)
- U2 pad 3: Net-(U1-Pad1) -> (no net)
- U2 pad 4: Net-(U1-Pad3) -> (no net)
- U2 pad 5: Net-(U2-Pad5) -> (no net)
- U2 pad 6: Net-(U2-Pad6) -> (no net)
- U2 pad 7: Net-(U2-Pad7) -> (no net)
- microcontroller1 pad 1: Net-(microcontroller1-Pad1) -> (no net)
- microcontroller1 pad 10: Net-(microcontroller1-Pad10) -> (no net)
- microcontroller1 pad 11: Net-(microcontroller1-Pad11) -> (no net)
- microcontroller1 pad 12: Net-(microcontroller1-Pad12) -> (no net)
- microcontroller1 pad 13: Net-(microcontroller1-Pad13) -> (no net)
- microcontroller1 pad 14: Net-(microcontroller1-Pad14) -> (no net)
- microcontroller1 pad 15: Net-(microcontroller1-Pad15) -> (no net)
- microcontroller1 pad 16: Net-(microcontroller1-Pad16) -> (no net)
- microcontroller1 pad 17: Net-(microcontroller1-Pad17) -> (no net)
- microcontroller1 pad 18: Net-(microcontroller1-Pad18) -> (no net)
- microcontroller1 pad 19: Net-(microcontroller1-Pad19) -> (no net)
- microcontroller1 pad 20: Net-(microcontroller1-Pad20) -> (no net)
- microcontroller1 pad 21: Net-(microcontroller1-Pad21) -> (no net)
- microcontroller1 pad 22: Net-(microcontroller1-Pad22) -> (no net)
- microcontroller1 pad 23: Net-(microcontroller1-Pad23) -> (no net)
- microcontroller1 pad 24: Net-(microcontroller1-Pad24) -> (no net)
- microcontroller1 pad 25: Net-(microcontroller1-Pad25) -> (no net)
- microcontroller1 pad 26: Net-(microcontroller1-Pad26) -> (no net)
- microcontroller1 pad 27: Net-(microcontroller1-Pad27) -> (no net)
- microcontroller1 pad 28: Net-(microcontroller1-Pad28) -> (no net)
- microcontroller1 pad 29: Net-(microcontroller1-Pad29) -> (no net)
- microcontroller1 pad 32: Net-(microcontroller1-Pad32) -> (no net)
- microcontroller1 pad 33: Net-(microcontroller1-Pad33) -> (no net)
- microcontroller1 pad 34: Net-(microcontroller1-Pad34) -> (no net)
- microcontroller1 pad 35: Net-(microcontroller1-Pad35) -> (no net)
- microcontroller1 pad 36: Net-(microcontroller1-Pad36) -> (no net)
- microcontroller1 pad 37: Net-(microcontroller1-Pad37) -> (no net)
- microcontroller1 pad 38: Net-(microcontroller1-Pad38) -> (no net)
- microcontroller1 pad 39: Net-(microcontroller1-Pad39) -> Net-(U1-Pad2)
- microcontroller1 pad 4: Net-(microcontroller1-Pad4) -> (no net)
- microcontroller1 pad 40: Net-(microcontroller1-Pad40) -> (no net)
- microcontroller1 pad 41: Net-(microcontroller1-Pad41) -> (no net)
- microcontroller1 pad 42: Net-(microcontroller1-Pad42) -> (no net)
- microcontroller1 pad 43: Net-(U1-Pad1) -> (no net)
- microcontroller1 pad 44: Net-(U1-Pad3) -> (no net)
- microcontroller1 pad 45: Net-(microcontroller1-Pad45) -> Net-(R2-Pad1)
- microcontroller1 pad 46: Net-(microcontroller1-Pad46) -> Net-(R1-Pad2)
- microcontroller1 pad 47: Net-(microcontroller1-Pad47) -> (no net)
- microcontroller1 pad 48: Net-(microcontroller1-Pad48) -> (no net)
- microcontroller1 pad 49: Net-(microcontroller1-Pad49) -> (no net)
- microcontroller1 pad 5: Net-(microcontroller1-Pad5) -> (no net)
- microcontroller1 pad 50: Net-(microcontroller1-Pad50) -> (no net)
- microcontroller1 pad 51: Net-(microcontroller1-Pad51) -> Net-(R1-Pad1)
- microcontroller1 pad 52: Net-(U1-Pad4) -> (no net)
- microcontroller1 pad 54: Net-(microcontroller1-Pad54) -> (no net)
- microcontroller1 pad 55: Net-(microcontroller1-Pad55) -> (no net)
- microcontroller1 pad 56: Net-(microcontroller1-Pad56) -> (no net)
- microcontroller1 pad 57: Net-(microcontroller1-Pad57) -> (no net)
- microcontroller1 pad 6: Net-(microcontroller1-Pad6) -> (no net)
- microcontroller1 pad 7: Net-(microcontroller1-Pad7) -> (no net)
- microcontroller1 pad 8: Net-(microcontroller1-Pad8) -> (no net)
- microcontroller1 pad 9: Net-(microcontroller1-Pad9) -> (no net)
Routing:
- net Net-(R1-Pad1): track 0.00 -> 74.1 mm
- net Net-(C3-Pad1): track 0.00 -> 72.0 mm
- net Net-(Battery2-Pad2): track 0.00 -> 58.7 mm
- net Net-(U1-Pad2): track 0.00 -> 58.1 mm
- net Net-(U3-Pad3): track 69.6 -> 23.3 mm
- net Net-(U3-Pad2): track 66.7 -> 21.0 mm
- net (no net): track 0.00 -> 39.1 mm
- net Net-(RF1-Pad9): track 27.4 -> 61.4 mm
- net Net-(RF1-Pad7): track 27.4 -> 61.4 mm
- net Net-(R1-Pad2): track 0.00 -> 31.5 mm
- net Net-(U1-Pad4): track 31.4 -> 0.00 mm
- net Net-(R2-Pad1): track 0.00 -> 29.1 mm
- net Net-(Battery1-Pad2): track 107.2 -> 80.7 mm
- net Net-(C2-Pad1): track 116.0 -> 89.6 mm
- net Net-(U1-Pad1): track 23.4 -> 0.00 mm
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
Commit message: update
Parts:
- added Battery2: 9V, Mounting Holes:1x02, F.Cu at (196.8, 91.4)
- added C4: 0.33uF, Capacitor_SMD:CP_Elec_3x5.3, F.Cu at (201.6, 86.8)
- GPS1: renamed from U3; footprint Connector_PinSocket_2.54mm:PinSocket_1x04_P2.54mm_Vertical -> Connector_PinHeader_1.00mm:PinHeader_1x04_P1.00mm_Horizontal
- renumbered U1 to ACCEL1, U2 to barometer1
Connections:
- linear_volt_reg2 pad 1: (no net) -> Net-(Battery2-Pad1)
Routing:
- net Net-(R1-Pad1): track 0.00 -> 74.1 mm
- net Net-(ACCEL1-Pad5): track 74.1 -> 0.00 mm

Commit message: update
Parts:
- GPS1: footprint Connector_PinHeader_1.00mm:PinHeader_1x04_P1.00mm_Horizontal -> Connector_PinSocket_1.00mm:PinSocket_1x04_P1.00mm_Vertical
- R1, R2: footprint Resistors:0603 -> Resistor_THT:R_Axial_DIN0204_L3.6mm_D1.6mm_P5.08mm_Horizontal
- moved Battery1 112.9 mm to (236.2, 86.4), turned to 0 degrees
- moved C1 89.9 mm to (218.4, 91.4), turned to 90 degrees
- moved C2 84.6 mm to (227.3, 82.5)
- moved linear_volt_reg1 78.5 mm to (208.3, 80.0), turned to 90 degrees
- moved C3 72.2 mm to (139.7, 104.1), turned to 270 degrees
- moved C4 68.7 mm to (139.7, 116.6), turned to 270 degrees
- moved Battery2 63.9 mm to (135.9, 110.5), turned to 90 degrees
- moved linear_volt_reg2 54.6 mm to (148.6, 111.8)
- moved microcontroller1 35.5 mm to (179.1, 109.2), turned to 270 degrees
- moved R1 13.5 mm to (194.3, 105.4), turned to 0 degrees
- moved barometer1 13.0 mm to (201.9, 127.0)
- moved ACCEL1 12.6 mm to (194.3, 97.8), turned to 270 degrees
- moved R2 11.4 mm to (217.2, 102.9)
- turned GPS1 to 90 degrees
Routing:
- net Net-(C2-Pad1): track 89.6 -> 0.00 mm
- net Net-(Battery1-Pad2): track 80.7 -> 0.00 mm
- net Net-(R1-Pad1): track 74.1 -> 0.00 mm
- net Net-(C3-Pad1): track 72.0 -> 0.00 mm
- net Net-(RF1-Pad9): track 61.4 -> 0.00 mm
- net Net-(RF1-Pad7): track 61.4 -> 0.00 mm
- net Net-(Battery2-Pad2): track 58.7 -> 0.00 mm
- net Net-(ACCEL1-Pad2): track 58.1 -> 0.00 mm
- net (no net): track 39.1 -> 6.91 mm
- net Net-(ACCEL1-Pad1): track 31.5 -> 0.00 mm
- net Net-(ACCEL1-Pad3): track 29.1 -> 0.00 mm
- net Net-(GPS1-Pad3): track 23.3 -> 0.43 mm
- net Net-(GPS1-Pad2): track 21.0 -> 0.00 mm
- net Net-(Battery1-Pad1): track 19.6 -> 0.00 mm
